Commit message: built depth_camera

File: src/Firmware/Tools/sitl_gazebo/models/rotors_description/urdf/iris.xacro (robot description, xacro)
@@ -137,3 +137,10 @@
     <xacro:insert_block name="rotor_inertia" />
   </xacro:vertical_rotor>
+  <link name="teratower">
+   <visual>
+    <geometry>
+      <mesh filename="package://pkg/m.dae"/>
+    </geometry>
+  </visual>
+  </link>
 </robot>

File: src/Firmware/Tools/sitl_gazebo/models/rotors_description/urdf/iris_base.xacro (robot description, xacro)
@@ -178,3 +178,41 @@
     </xacro:bag_plugin_macro>
   </xacro:if>
+<!-- Teraranger tower -->
+<gazebo reference="base_ir_front">
+   <sensor type="ray" name="TeraRanger">
+      <pose>0 0 0 0 0 0</pose>
+      <visualize>true</visualize>
+      <update_rate>20</update_rate>
+      <ray>
+         <scan>
+            <horizontal>
+               <samples>10</samples>
+               <resolution>1</resolution>
+               <min_angle>-0.14835</min_angle>
+               <max_angle>0.14835</max_angle>
+            </horizontal>
+            <vertical>
+               <samples>10</samples>
+               <resolution>1</resolution>
+               <min_angle>-0.14835</min_angle>
+               <max_angle>0.14835</max_angle>
+            </vertical>
+         </scan>
+         <range>
+            <min>0.01</min>
+            <max>2</max>
+            <resolution>0.02</resolution>
+         </range>
+      </ray>
+      <plugin filename="libgazebo_ros_range.so" name="gazebo_ros_range">
+         <gaussianNoise>0.005</gaussianNoise>
+         <alwaysOn>true</alwaysOn>
+         <updateRate>50</updateRate>
+         <topicName>sensor/ir_front</topicName>
+         <frameName>base_ir_front</frameName>
+         <radiation>INFRARED</radiation>
+         <fov>0.2967</fov>
+      </plugin>
+   </sensor>
+   </gazebo>
 </robot>

File: src/Firmware/Tools/sitl_gazebo/models/teraranger_tower/teraranger_tower.urdf (robot description, URDF)
Before this commit: robot teraranger_tower.urdf, 1 links, 0 joints
Links:
- link base_link: geometry collision box size=0.1 0.1 0.1; visual mesh 
